File: pcb/logic_handle.kicad_pcb (KiCad board)
At the start: 2 copper layers, 100 x 35 mm, 60 parts, among them J1 Conn_01x05_Male, Q1 BSS214NW, SW1 SW_Push, U1 NCP1117-3.3_TO252, U2 TXS0108EPW, U3 MSP430FR5739IDAR, Y1 Crystal

Commit message: [WIP]: Finish logic PCB
Parts:
- moved TP2 6.35 mm to (68.7, 2.03)
Routing:
- net +3V3: track 103.3 -> 113.5 mm
Other:
- board text added: "3V3"
- board text added: "BTN"
- board text added: "IC_BTN"
- board text added: "IC_LED"
- board text added: "IO ALTERNATIVES"
- board text added: "JLCJLCJLCJLC"
- board text added: "LED"
- board text added: "LEVEL SHIFT BYPASS"
- board text added: "LitePog Logic Board Rev 1"
- board text added: "NPX"
- board text added: "NPX_BPS"
- board text added: "NPX_CLK"
- board text added: "NPX_CLK_AUX"
- board text added: "SHFT_EN"
- board text added: "VCC"
