File: pcb/programmer_converter.kicad_pcb (KiCad board)
At the start: 2 copper layers, 41.9 x 25.4 mm, 15 parts, among them J1 Conn_01x06_Female, J2 Conn_01x05_Male, J3 Conn_01x05_Male, J4 Conn_01x06_Male

Commit message: programmer_converter: Add serial number locator for JLCPCB (#5)
Other:
- board text added: "JLCJLCJLCJLC"
