File: pcb/programmer_converter.sch (KiCad schematic (older format))
At the start: 15 parts, among them J1 Conn_01x06_Female, J2 Conn_01x05_Male, J3 Conn_01x05_Male, J4 Conn_01x06_Male

Commit message: pcb: Cleanup BOM items (#7)
Replaced out of stock components with substitutes
Parts:
- J1: Digikey (none) -> 1212-1351-ND
- J4: Digikey (none) -> 1849-PR20B06HBNN-ND
Changed lines of the file:
@@
 F 1 "Conn_01x06_Female" H 6728 3035 50  0000 L CNN
 F 2 "Gigahawk:851-87-006-20-001101" H 6700 3150 50  0001 C CNN
-F 3 "~" H 6700 3150 50  0001 C CNN
+F 3 "https://www.precidip.com/AppHost/9696,1/Scripts/Modules/Catalog/Default.aspx?c=7&i=204&p=80&pdf=1&dsku=851-PP-NNN-20-001101" H 6700 3150 50  0001 C CNN
+F 4 "1212-1351-ND" H 6700 3150 50  0001 C CNN "Digikey"
 	1    6700 3150
 	1    0    0    -1
@@
 F 1 "Conn_01x06_Male" H 4058 3440 50  0000 C CNN
 F 2 "Connector_PinHeader_1.27mm:PinHeader_1x06_P1.27mm_Horizontal" H 3950 3150 50  0001 C CNN
-F 3 "~" H 3950 3150 50  0001 C CNN
+F 3 "https://media.metz-connect.com/files/171/Data_sheet_PR20BXXHBNN.PDF" H 3950 3150 50  0001 C CNN
+F 4 "1849-PR20B06HBNN-ND" H 3950 3150 50  0001 C CNN "Digikey"
 	1    3950 3150
 	-1   0    0    -1
